File: hardware/observer/rev_d/observer.brd (EAGLE design)
At the start: 49.5 x 60.2 mm, 62 parts, among them J1 CON_HEADER_2X05-SMD+SHROUDED, J2 CON_HEADER_2X05-SMD+SHROUDED, J3 TC2030-CC2538-BL-NL, J4 JUMPER-PTH-2-NO, J5 PINHD-2X8/SMD, J6 CON_HEADER_2X05-PTH+SHROUDED_A, P9/P8 BBB_HEADER, U1 LPS331AP, U10 TPS62740, U11 DMG1013UW-7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

Commit message: rev_d gerbers
Parts:
- removed LOGO2: UMICH_SOLID_TINY, logos:UMICH_SOLID_50MIL
- added U$2: (no value), logos:UMICH_SOLID_50MIL
- moved R11 0.57 mm to (37.8, 23.9)
Routing:
- net LIGHT_INT: track 36.0 -> 37.4 mm, vias 2 -> 3
- net VCC: track 278.9 -> 279.6 mm
- net GND: vias 41 -> 42
Changed lines of the file:
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@@
 <attribute name="VALUE" x="30.734" y="42.672" size="1.016" layer="27" font="vector" ratio="12" rot="R180" align="bottom-center"/>
 </element>
-<element name="LOGO2" library="logos" package="UMICH_SOLID_50MIL" value="UMICH_SOLID_TINY" x="26.416" y="59.309"/>
 <element name="P9/P8" library="observer" package="BBB_HEADERS" value="BBB_HEADER" x="0.762" y="0.762" smashed="yes">
 <attribute name="VALUE" x="0.762" y="59.817" size="1.27" layer="27" font="vector"/>
@@
 </element>
 <element name="U11" library="pfet" package="SOT-323" value="DMG1013UW-7" x="46.736" y="12.192" rot="R180"/>
-<element name="R11" library="passives" package="0402_RES" value="10k" x="38.354" y="23.622" smashed="yes" rot="R90">
-<attribute name="DIGIKEY" value="RHM30CECT-ND" x="38.354" y="23.622" size="1.778" layer="27" rot="R90" display="off"/>
-<attribute name="NAME" x="37.211" y="23.876" size="0.8128" layer="25" font="vector" ratio="12" rot="R270" align="bottom-center"/>
-<attribute name="VALUE" x="39.751" y="23.622" size="1.016" layer="27" font="vector" ratio="12" rot="R90" align="bottom-center"/>
+<element name="R11" library="passives" package="0402_RES" value="10k" x="37.846" y="23.876" smashed="yes" rot="R90">
+<attribute name="DIGIKEY" value="RHM30CECT-ND" x="37.846" y="23.876" size="1.778" layer="27" rot="R90" display="off"/>
+<attribute name="NAME" x="36.703" y="24.13" size="0.8128" layer="25" font="vector" ratio="12" rot="R270" align="bottom-center"/>
+<attribute name="VALUE" x="39.243" y="23.876" size="1.016" layer="27" font="vector" ratio="12" rot="R90" align="bottom-center"/>
 </element>
 <element name="U$1" library="logos" package="UMICH_SOLID_75MIL" value="" x="40.132" y="11.43"/>
+<element name="U$2" library="logos" package="UMICH_SOLID_50MIL" value="" x="26.416" y="59.436"/>
 </elements>
 <signals>
@@
 <wire x1="17.78" y1="9.144" x2="18.542" y2="9.906" width="0.254" layer="1"/>
 <contactref element="R11" pad="2"/>
-<wire x1="38.354" y1="24.05506875" x2="40.894" y2="24.05506875" width="0.254" layer="1"/>
-<wire x1="40.894" y1="24.05506875" x2="41.58106875" y2="23.368" width="0.254" layer="1"/>
+<wire x1="37.846" y1="24.30906875" x2="40.894" y2="24.30906875" width="0.254" layer="1"/>
+<wire x1="40.894" y1="24.30906875" x2="41.58106875" y2="23.368" width="0.254" layer="1"/>
 <wire x1="45.39106875" y1="21.59" x2="45.466" y2="21.51506875" width="0" layer="19" extent="1-1"/>
 </signal>
@@
 <wire x1="12.192" y1="11.672" x2="12.192" y2="11.684" width="0.254" layer="1"/>
 <via x="14.097" y="12.065" extent="1-16" drill="0.254"/>
-<wire x1="39.6494" y1="19.88946875" x2="40.64" y2="23.114" width="0" layer="19" extent="1-1"/>
+<via x="35.433" y="8.636" extent="1-16" drill="0.254"/>
 </signal>
 <signal name="N$3">
@@
 <wire x1="27.488" y1="23.576" x2="27.488" y2="22.042" width="0.254" layer="16"/>
 <wire x1="27.488" y1="22.042" x2="28.448" y2="21.082" width="0.254" layer="16"/>
-<wire x1="28.448" y1="21.082" x2="37.084" y2="21.082" width="0.254" layer="16"/>
+<wire x1="28.448" y1="21.082" x2="34.036" y2="21.082" width="0.254" layer="16"/>
+<wire x1="34.036" y1="21.082" x2="37.084" y2="21.082" width="0.254" layer="16"/>
 <wire x1="37.084" y1="21.082" x2="38.354" y2="19.812" width="0.254" layer="16"/>
 <via x="38.354" y="19.812" extent="1-16" drill="0.254"/>
@@
 <wire x1="38.542" y1="19.624" x2="38.542" y2="18.657" width="0.254" layer="1"/>
 <contactref element="R11" pad="1"/>
-<wire x1="38.354" y1="23.18893125" x2="38.354" y2="19.812" width="0.254" layer="1"/>
+<wire x1="37.846" y1="23.44293125" x2="36.39693125" y2="23.44293125" width="0.254" layer="1"/>
+<wire x1="36.39693125" y1="23.44293125" x2="34.036" y2="21.082" width="0.254" layer="1"/>
+<via x="34.036" y="21.082" extent="1-16" drill="0.254"/>
 </signal>
 <signal name="N$4">
@@
 <wire x1="31.75" y1="11.25093125" x2="31.67506875" y2="11.176" width="0.254" layer="1"/>
 <wire x1="30.80893125" y1="17.018" x2="30.80893125" y2="16.002" width="0.254" layer="1"/>
-<wire x1="30.80893125" y1="16.002" x2="30.2895" y2="15.48256875" width="0.254" layer="1"/>
-<wire x1="30.2895" y1="15.48256875" x2="30.2895" y2="14.2875" width="0.254" layer="1"/>
+<wire x1="30.80893125" y1="16.002" x2="30.2895" y2="15.73656875" width="0.254" layer="1"/>
+<wire x1="30.2895" y1="15.73656875" x2="30.2895" y2="14.2875" width="0.254" layer="1"/>
 <wire x1="30.2895" y1="14.2875" x2="31.2119" y2="13.3651" width="0.254" layer="1"/>
 <wire x1="31.2119" y1="13.3651" x2="31.2119" y2="13.274" width="0.254" layer="1"/>
